File: PlasticBottleRecycler-pcb.kicad_sch (KiCad schematic)
At the start: 35 parts, among them J1 SWIM, J2 LCD, J3 Screw_Terminal_01x04, J4 NTC, J5 HEATER, J6 FAN1, J7 +12V, J8 +5V, Q1 IRF3205, Q2 BC337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

Commit message: Add PCB design
Parts:
- removed D1, D2: LED, symbol Device:LED
- removed R10, R8: 470, symbol Device:R
- C1: footprint (none) -> Capacitor_THT:CP_Radial_D10.0mm_P5.00mm
- C2, C3, C5: footprint (none) -> Capacitor_THT:C_Disc_D6.0mm_W2.5mm_P5.00mm
- C4: footprint (none) -> Capacitor_THT:CP_Radial_D4.0mm_P2.00mm
- J1: footprint (none) -> Connector_PinHeader_2.54mm:PinHeader_1x04_P2.54mm_Vertical
- J2: footprint (none) -> Connector_PinHeader_2.54mm:PinHeader_1x10_P2.54mm_Vertical
- J3: footprint (none) -> TerminalBlock:TerminalBlock_bornier-4_P5.08mm
- J4: footprint (none) -> Connector_JST:JST_XH_B2B-XH-A_1x02_P2.50mm_Vertical
- J5, J7, J8: footprint (none) -> TerminalBlock:TerminalBlock_bornier-2_P5.08mm
- J6: footprint (none) -> Connector_PinHeader_2.54mm:PinHeader_1x02_P2.54mm_Vertical
- R1, R2, R3, R4, R5, R6, R7: footprint (none) -> Resistor_THT:R_Axial_DIN0204_L3.6mm_D1.6mm_P5.08mm_Horizontal
- R8: renamed from R9; footprint (none) -> Resistor_THT:R_Axial_DIN0207_L6.3mm_D2.5mm_P10.16mm_Horizontal
- RV1: value 1K -> 100K; footprint (none) -> Potentiometer_THT:Potentiometer_Vishay_T73YP_Vertical
- SW1, SW2, SW3, SW4: footprint (none) -> Button_Switch_THT:SW_PUSH_6mm_H5mm
- U1: footprint (none) -> Package_QFP:LQFP-32_7x7mm_P0.8mm
Connections:
- net +12V: now also C1.1, J7.2 (Pin_2); no longer J7.1 (Pin_1)
- net +5V: now also J8.2 (Pin_2); no longer J8.1 (Pin_1)
- net A4988_DIR: now also U1.24 (SPI_MISO/PC7); no longer U1.18 (PC1/TIM1_CH1/UART2_CLK)
- net A4988_ENA: now also U1.18 (PC1/TIM1_CH1/UART2_CLK); no longer U1.24 (SPI_MISO/PC7)
- net A4988_MS1: now also U1.19 (PC2/TIM1_CH2); no longer U1.23 (SPI_MOSI/PC6)
- net A4988_MS2: now also U1.20 (PC3/TIM1_CH3); no longer U1.22 (SPI_SCK/PC5)
- net A4988_MS3: now also U1.22 (SPI_SCK/PC5); no longer U1.21 (PC4/TIM1_CH4)
- net A4988_SLP: now also U1.23 (SPI_MOSI/PC6); no longer U1.20 (PC3/TIM1_CH3)
- net A4988_STP: now also U1.21 (PC4/TIM1_CH4); no longer U1.19 (PC2/TIM1_CH2)
- net GND: now also C4.2, J7.1 (Pin_1), J8.1 (Pin_1); no longer J8.2 (Pin_2)
- net at R6.2, R7.1, U2.1 (ADJ): no longer C4.2
Other:
- moved on the sheet: C1
